File: sr-jv-esp32.kicad_pcb (KiCad board)
At the start: 4 copper layers, 58.5 x 85.5 mm, 80 parts, among them J1 Conn_40_SRJV_MountingPin, J2 USB_C_Receptacle_USB2.0_14P, J3 Conn_01x06, J4 Conn_01x02, Q1 2N7002, SW1 TS-1187A, U1 AMS1117-3.3, U10 SN74HCS595, U11 SN74HCS595, U12 SN74HCS595, U13 NOR_FLASH_29064, U2 DNP/MAX809S, U3 ESP32-S3-WROOM-1, U4 74HC86, U5 74HC08, U6 SN74LVC8T245, U7 SN74LVC8T245, U8 SN74LVC8T245, U9 SN74LVC8T245

Commit message: Upload MP 1.2 version
Parts:
- removed D4: DNP/1N4148W, Diode_SMD:D_SOD-123
- added C29: 100n, Capacitor_SMD:C_0603_1608Metric, B.Cu at (7.50, 58.0)
- added R27: 10K, Resistor_SMD:R_0603_1608Metric, B.Cu at (4.30, 74.2)
- added U14: SN74LVC1G125DBV, Package_TO_SOT_SMD:SOT-23-5, B.Cu at (4.00, 55.1)
- added U15: SN74LVC1G125DBV, Package_TO_SOT_SMD:SOT-23-5, B.Cu at (9.00, 61.0)
- added U16: SN74LVC1G125DBV, Package_TO_SOT_SMD:SOT-23-5, B.Cu at (4.00, 61.0)
- R1: value DNP/1k -> DNP
- R15, R19: value DNP/10k -> DNP
- U10, U11, U12: value SN74HCS595 -> SN74AHC595
- U4: value 74HC86 -> 74AHC86
- U5: value 74HC08 -> SN74LVC1G125DBV; footprint Package_SO:TSSOP-14_4.4x5mm_P0.65mm -> Package_TO_SOT_SMD:SOT-23-5
- moved U5 3.32 mm to (9.00, 55.1)
- moved U4 3.03 mm to (6.40, 68.0)
- moved C12 3.00 mm to (6.00, 64.0)
- moved C11 1.14 mm to (7.10, 52.2)
- moved R15 0.70 mm to (56.3, 68.6)
- moved R16 0.70 mm to (56.3, 70.5)
- moved R18 0.70 mm to (56.3, 75.0)
- moved R19 0.70 mm to (56.3, 73.0)
Connections:
- U4 pad 10: /CE# -> GND
- U4 pad 11: /~{EXP_OE_5V} -> unconnected-(U4-Pad11)
- U4 pad 12: Net-(U4-Pad12) -> GND
- U4 pad 13: Net-(U4-Pad13) -> GND
- U4 pad 8: Net-(U4-Pad13) -> unconnected-(U4-Pad8)
- U4 pad 9: /~{WOE} -> GND
- U5 pad 2: /CE1# -> /~{WOE}
- U5 pad 3: Net-(U5-Pad10) -> GND
- U5 pad 4: /CE2# -> /~{EXP_OE_5V}
- U5 pad 5: /CE3# -> +5V
Routing:
- net /CE#: track 64.6 -> 0.00 mm, vias 6 -> 0
- net +5V: track 400.6 -> 453.2 mm, vias 15 -> 19
- net /WA22: track 91.2 -> 57.8 mm, vias 6 -> 4
- net /WA21: track 92.8 -> 61.0 mm, vias 6 -> 4
- net /~{EXP_OE_5V}: track 63.9 -> 78.7 mm, vias 4 -> 5
- net /~{CE_FLASH}: track 106.1 -> 93.9 mm, vias 5 -> 4
- net /~{WOE}: track 33.8 -> 45.6 mm, vias 2 -> 7
- net Net-(U4-Pad12): track 10.5 -> 0.00 mm, vias 2 -> 0
- net /CE3#: track 40.4 -> 49.0 mm
- net Net-(U4-Pad13): track 6.53 -> 0.00 mm, vias 2 -> 0
- net Net-(U5-Pad10): track 6.26 -> 0.00 mm
- net Net-(U5-Pad6): track 5.73 -> 0.00 mm
- net /CE1#: track 37.3 -> 42.6 mm
- net /CE2#: track 35.9 -> 40.5 mm
- net /CE0#: track 20.1 -> 18.7 mm
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Other:
- board text added: "28 FEB. 2025 REV: 1.2"
- board text removed: "24 FEB. 2025 REV: 1.1"
