File: sr-jv-esp32.kicad_sch (KiCad schematic)
At the start: 80 parts, among them J1 Conn_40_SRJV_MountingPin, J2 USB_C_Receptacle_USB2.0_14P, J3 Conn_01x06, J4 Conn_01x02, Q1 2N7002, SW1 TS-1187A, U1 AMS1117-3.3, U10 SN74HCS595, U11 SN74HCS595, U12 SN74HCS595, U13 NOR_FLASH_29064, U2 DNP/MAX809S, U3 ESP32-S3-WROOM-1, U4 74HC86, U5 74HC08, U6 SN74LVC8T245, U7 SN74LVC8T245, U8 SN74LVC8T245, U9 SN74LVC8T245

Commit message: Upload MP 1.2 version
Parts:
- removed D4: DNP/1N4148W, Diode_SMD:D_SOD-123, symbol Device:D
- removed U5: 74HC08, Package_SO:TSSOP-14_4.4x5mm_P0.65mm, symbol 74xx:74LS08
- added C29: 100n, Capacitor_SMD:C_0603_1608Metric, symbol Device:C_Small
- added R27: 10K, Resistor_SMD:R_0603_1608Metric, symbol Device:R
- added U14, U15, U16, U5: SN74LVC1G125DBV, Package_TO_SOT_SMD:SOT-23-5, symbol 74xGxx:SN74LVC1G125DBV
- C6: value 100uF/10v -> 220uF/6.3v
- R1: value DNP/1k -> DNP
- R15, R19: value DNP/10k -> DNP
- U10, U11, U12: value SN74HCS595 -> SN74AHC595
- U4: value 74HC86 -> 74AHC86
Connections:
- net CE# is gone; now on net GND: U4.10
- net +5V: now also C29.1, R27.1, U14.5 (VCC), U15.5 (VCC), U16.5 (VCC), U5.5 (VCC)
- net CE0#: now also U5.1
- net CE1#: now also U14.1
- net CE2#: now also U15.1
- net CE3#: now also U16.1
- net GND: now also U4.12, U4.13, U4.9, C29.2, U14.3 (GND), U15.3 (GND), U16.3 (GND), U5.3 (GND)
- net ~{EXP_OE_5V}: now also R27.2, U14.4, U15.4, U16.4, U5.4; no longer U4.11
- net ~{WOE}: now also U14.2, U15.2, U16.2, U5.2; no longer U4.9
- net at U4.8: no longer U4.13
Other:
- note added: "OR 74LV86"
- note removed: "ONE OF ANY CE LOW WILL OUTPUT LOW ALL CE HIGH WILL OUTPUT HIGH"
- moved on the sheet: C11, C27, C7, D1, R1, R2, R24, U2, U4C, U4D
